File: KiCad/InterConn.kicad_sch (KiCad schematic)
At the start: 5 parts

Commit message: created
Connections:
- new net SCL: ExtensionBoard.3 (Pin_3)
- new net SDA: ExtensionBoard.1 (Pin_1)
- now unconnected: ExtensionBoard.5 (Pin_5), ExtensionBoard.7 (Pin_7), ExtensionBoard.9 (Pin_9)
Changed lines of the file:
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@@
   (junction (at 97.79 101.6) (diameter 0) (color 0 0 0 0)
   )
-  (junction (at 118.11 82.55) (diameter 0) (color 0 0 0 0)
-  )
   (junction (at 134.62 52.07) (diameter 0) (color 0 0 0 0)
   )
@@
   (junction (at 100.33 101.6) (diameter 0) (color 0 0 0 0)
   )
-  (junction (at 115.57 82.55) (diameter 0) (color 0 0 0 0)
-  )
   (junction (at 115.57 101.6) (diameter 0) (color 0 0 0 0)
   )
@@
   (junction (at 100.33 68.58) (diameter 0) (color 0 0 0 0)
   )
-  (junction (at 113.03 82.55) (diameter 0) (color 0 0 0 0)
-  )
   (junction (at 118.11 101.6) (diameter 0) (color 0 0 0 0)
   )
@@
     (stroke (width 0) (type default))
   )
+  (wire (pts (xy 102.87 66.04) (xy 102.87 85.09))
+    (stroke (width 0) (type default))
+  )
   (wire (pts (xy 134.62 52.07) (xy 134.62 50.8))
     (stroke (width 0) (type default))
   )
-  (wire (pts (xy 120.65 82.55) (xy 120.65 85.09))
+  (wire (pts (xy 120.65 81.28) (xy 120.65 85.09))
     (stroke (width 0) (type default))
   )
@@
     (stroke (width 0) (type default))
   )
-  (wire (pts (xy 118.11 82.55) (xy 120.65 82.55))
-    (stroke (width 0) (type default))
-  )
   (wire (pts (xy 120.65 101.6) (xy 120.65 97.79))
     (stroke (width 0) (type default))
   )
-  (wire (pts (xy 102.87 85.09) (xy 102.87 68.58))
-    (stroke (width 0) (type default))
-  )
   (wire (pts (xy 95.25 55.88) (xy 115.57 55.88))
     (stroke (width 0) (type default))
@@
     (stroke (width 0) (type default))
   )
+  (wire (pts (xy 120.65 81.28) (xy 128.905 81.28))
+    (stroke (width 0) (type default))
+  )
   (wire (pts (xy 90.17 80.01) (xy 92.71 80.01))
     (stroke (width 0) (type default))
@@
     (stroke (width 0) (type default))
   )
+  (wire (pts (xy 107.95 73.66) (xy 107.95 85.09))
+    (stroke (width 0) (type default))
+  )
   (wire (pts (xy 118.11 97.79) (xy 118.11 101.6))
     (stroke (width 0) (type default))
   )
-  (wire (pts (xy 107.95 76.2) (xy 125.73 76.2))
-    (stroke (width 0) (type default))
-  )
   (wire (pts (xy 118.11 101.6) (xy 120.65 101.6))
     (stroke (width 0) (type default))
@@
     (stroke (width 0) (type default))
   )
-  (wire (pts (xy 118.11 85.09) (xy 118.11 82.55))
+  (wire (pts (xy 118.11 77.47) (xy 118.11 85.09))
     (stroke (width 0) (type default))
   )
@@
     (stroke (width 0) (type default))
   )
+  (wire (pts (xy 125.73 66.04) (xy 102.87 66.04))
+    (stroke (width 0) (type default))
+  )
   (wire (pts (xy 115.57 59.69) (xy 134.62 59.69))
     (stroke (width 0) (type default))
   )
-  (wire (pts (xy 105.41 85.09) (xy 105.41 72.39))
-    (stroke (width 0) (type default))
-  )
   (wire (pts (xy 115.57 101.6) (xy 118.11 101.6))
     (stroke (width 0) (type default))
@@
     (stroke (width 0) (type default))
   )
+  (wire (pts (xy 118.11 77.47) (xy 128.905 77.47))
+    (stroke (width 0) (type default))
+  )
   (wire (pts (xy 90.17 72.39) (xy 97.79 72.39))
     (stroke (width 0) (type default))
   )
+  (wire (pts (xy 105.41 69.85) (xy 105.41 85.09))
+    (stroke (width 0) (type default))
+  )
   (wire (pts (xy 105.41 97.79) (xy 105.41 101.6))
     (stroke (width 0) (type default))
   )
-  (wire (pts (xy 102.87 68.58) (xy 125.73 68.58))
-    (stroke (width 0) (type default))
-  )
   (wire (pts (xy 113.03 97.79) (xy 113.03 101.6))
     (stroke (width 0) (type default))
@@
     (stroke (width 0) (type default))
   )
-  (wire (pts (xy 105.41 72.39) (xy 125.73 72.39))
+  (wire (pts (xy 125.73 73.66) (xy 107.95 73.66))
     (stroke (width 0) (type default))
   )
@@
     (stroke (width 0) (type default))
   )
-  (wire (pts (xy 110.49 82.55) (xy 113.03 82.55))
-    (stroke (width 0) (type default))
-  )
   (wire (pts (xy 92.71 101.6) (xy 95.25 101.6))
     (stroke (width 0) (type default))
@@
     (stroke (width 0) (type default))
   )
+  (wire (pts (xy 125.73 69.85) (xy 105.41 69.85))
+    (stroke (width 0) (type default))
+  )
   (wire (pts (xy 97.79 97.79) (xy 97.79 101.6))
     (stroke (width 0) (type default))
   )
-  (wire (pts (xy 115.57 82.55) (xy 118.11 82.55))
-    (stroke (width 0) (type default))
-  )
   (wire (pts (xy 97.79 59.69) (xy 97.79 72.39))
     (stroke (width 0) (type default))
@@
     (stroke (width 0) (type default))
   )
-  (wire (pts (xy 107.95 85.09) (xy 107.95 76.2))
-    (stroke (width 0) (type default))
-  )
-  (wire (pts (xy 113.03 82.55) (xy 115.57 82.55))
-    (stroke (width 0) (type default))
-  )
-  (global_label "GPIO32" (shape input) (at 125.73 68.58 0)
+  (global_label "SDA" (shape input) (at 128.905 81.28 0)
     (effects (font (size 1.27 1.27)) (justify left))
-    (property "Intersheetrefs" "${INTERSHEET_REFS}" (at 125.73 68.58 0)
+    (property "Intersheetrefs" "${INTERSHEET_REFS}" (at 128.905 81.28 0)
+      (effects (font (size 1.27 1.27)) hide)
+    )
+  )
+  (global_label "GPIO32" (shape input) (at 125.73 66.04 0)
+    (effects (font (size 1.27 1.27)) (justify left))
+    (property "Intersheetrefs" "${INTERSHEET_REFS}" (at 125.73 66.04 0)
+      (effects (font (size 1.27 1.27)) hide)
+    )
+  )
+  (global_label "SCL" (shape input) (at 128.905 77.47 0)
+    (effects (font (size 1.27 1.27)) (justify left))
+    (property "Intersheetrefs" "${INTERSHEET_REFS}" (at 128.905 77.47 0)
       (effects (font (size 1.27 1.27)) hide)
     )
@@
     )
   )
-  (global_label "GPIO15" (shape input) (at 125.73 76.2 0)
+  (global_label "GPIO15" (shape input) (at 125.73 73.66 0)
     (effects (font (size 1.27 1.27)) (justify left))
-    (property "Intersheetrefs" "${INTERSHEET_REFS}" (at 125.73 76.2 0)
-      (effects (font (size 1.27 1.27)) hide)
-    )
-  )
-  (global_label "GPIO33" (shape input) (at 125.73 72.39 0)
+    (property "Intersheetrefs" "${INTERSHEET_REFS}" (at 125.73 73.66 0)
+      (effects (font (size 1.27 1.27)) hide)
+    )
+  )
+  (global_label "GPIO33" (shape input) (at 125.73 69.85 0)
     (effects (font (size 1.27 1.27)) (justify left))
-    (property "Intersheetrefs" "${INTERSHEET_REFS}" (at 125.73 72.39 0)
+    (property "Intersheetrefs" "${INTERSHEET_REFS}" (at 125.73 69.85 0)
       (effects (font (size 1.27 1.27)) hide)
     )
@@
     (pin "9")
     (instances
-      (project "ESP32extention"
+      (project "InterConn"
         (path "/4973e3e7-48dc-4f4c-a353-a7d40b7094c7"
           (reference "ExtensionBoard") (unit 1)
@@
     (pin "1")
     (instances
-      (project "ESP32extention"
+      (project "InterConn"
         (path "/4973e3e7-48dc-4f4c-a353-a7d40b7094c7"
           (reference "#PWR?") (unit 1)
@@
     (pin "1")
     (instances
-      (project "ESP32extention"
+      (project "InterConn"
         (path "/4973e3e7-48dc-4f4c-a353-a7d40b7094c7"
           (reference "#PWR?") (unit 1)
@@
     (pin "2")
     (instances
-      (project "ESP32extention"
+      (project "InterConn"
         (path "/4973e3e7-48dc-4f4c-a353-a7d40b7094c7"
           (reference "R1") (unit 1)
@@
     (pin "2")
     (instances
-      (project "ESP32extention"
+      (project "InterConn"
         (path "/4973e3e7-48dc-4f4c-a353-a7d40b7094c7"
           (reference "R2") (unit 1)
@@
     (pin "2")
     (instances
-      (project "ESP32extention"
+      (project "InterConn"
         (path "/4973e3e7-48dc-4f4c-a353-a7d40b7094c7"
           (reference "R3") (unit 1)
@@
     (pin "2")
     (instances
-      (project "ESP32extention"
+      (project "InterConn"
         (path "/4973e3e7-48dc-4f4c-a353-a7d40b7094c7"
           (reference "R4") (unit 1)

Commit message: init
Parts:
- renumbered ExtensionBoard to InterConn
Changed lines of the file:
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@@
   (symbol (lib_id "Connector_Generic:Conn_02x12_Odd_Even") (at 107.95 90.17 270) (unit 1)
     (in_bom yes) (on_board yes) (dnp no)
-    (property "Reference" "ExtensionBoard" (at 122.682 90.2716 90)
+    (property "Reference" "InterConn" (at 122.682 90.2716 90)
       (effects (font (size 1.27 1.27)) (justify left))
     )
@@
       (project "InterConn"
         (path "/4973e3e7-48dc-4f4c-a353-a7d40b7094c7"
-          (reference "ExtensionBoard") (unit 1)
+          (reference "InterConn") (unit 1)
         )
       )
